File: eagle/MHI-SPI_v1.0withValues.brd (EAGLE design)
At the start: 69.4 x 39.4 mm, 44 parts, among them U1 TSR_1-2450

Commit message: values for R2/R4 added
Parts:
- R1, R3: value (none) -> 1k
- R2, R4: value (none) -> 3k3
Changed lines of the file:
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@@
 <?xml version="1.0" encoding="utf-8"?>
 <!DOCTYPE eagle SYSTEM "eagle.dtd">
-<eagle version="9.4.2">
+<eagle version="9.5.1">
 <drawing>
 <settings>
@@
 <attribute name="VALUE" x="19.558" y="28.067" size="1.4224" layer="27"/>
 </element>
-<element name="R1" library="rcl" library_urn="urn:adsk.eagle:library:334" package="VMTA55" package3d_urn="urn:adsk.eagle:package:26121/2" value="" x="36.83" y="16.51" smashed="yes">
+<element name="R1" library="rcl" library_urn="urn:adsk.eagle:library:334" package="VMTA55" package3d_urn="urn:adsk.eagle:package:26121/2" value="1k" x="36.83" y="16.51" smashed="yes">
 <attribute name="NAME" x="40.767" y="14.097" size="1.27" layer="25" ratio="10"/>
 <attribute name="SPICEPREFIX" value="R" x="36.83" y="16.51" size="1.778" layer="27" display="off"/>
 <attribute name="VALUE" x="33.655" y="15.875" size="1.27" layer="27" ratio="10"/>
 </element>
-<element name="R2" library="rcl" library_urn="urn:adsk.eagle:library:334" package="VMTA55" package3d_urn="urn:adsk.eagle:package:26121/2" value="" x="54.61" y="16.51" smashed="yes">
+<element name="R2" library="rcl" library_urn="urn:adsk.eagle:library:334" package="VMTA55" package3d_urn="urn:adsk.eagle:package:26121/2" value="3k3" x="54.61" y="16.51" smashed="yes">
 <attribute name="NAME" x="48.641" y="14.097" size="1.27" layer="25" ratio="10"/>
 <attribute name="SPICEPREFIX" value="R" x="54.61" y="16.51" size="1.778" layer="27" display="off"/>
 <attribute name="VALUE" x="51.435" y="15.875" size="1.27" layer="27" ratio="10"/>
 </element>
-<element name="R3" library="rcl" library_urn="urn:adsk.eagle:library:334" package="VMTA55" package3d_urn="urn:adsk.eagle:package:26121/2" value="" x="36.83" y="20.32" smashed="yes">
+<element name="R3" library="rcl" library_urn="urn:adsk.eagle:library:334" package="VMTA55" package3d_urn="urn:adsk.eagle:package:26121/2" value="1k" x="36.83" y="20.32" smashed="yes">
 <attribute name="NAME" x="40.894" y="17.907" size="1.27" layer="25" ratio="10"/>
 <attribute name="SPICEPREFIX" value="R" x="36.83" y="20.32" size="1.778" layer="27" display="off"/>
 <attribute name="VALUE" x="33.655" y="19.685" size="1.27" layer="27" ratio="10"/>
 </element>
-<element name="R4" library="rcl" library_urn="urn:adsk.eagle:library:334" package="VMTA55" package3d_urn="urn:adsk.eagle:package:26121/2" value="" x="54.61" y="20.32" smashed="yes" rot="R180">
+<element name="R4" library="rcl" library_urn="urn:adsk.eagle:library:334" package="VMTA55" package3d_urn="urn:adsk.eagle:package:26121/2" value="3k3" x="54.61" y="20.32" smashed="yes" rot="R180">
 <attribute name="NAME" x="50.673" y="19.304" size="1.27" layer="25" ratio="10" rot="R180"/>
 <attribute name="SPICEPREFIX" value="R" x="54.61" y="20.32" size="1.778" layer="27" rot="R180" display="off"/>
